Commit message: Can generate rod link world. Rod joints not stable

File: Tools/simulation/gz/models/cable_rod/model.urdf (robot description, URDF)
Before this commit: robot tether, 3 links, 2 joints
Links:
- added link element_p1, mass 0.0001; visual cylinder length=0.0001 radius=0.01
- added link element_p2, mass 0.0001; visual cylinder length=0.0001 radius=0.01
- added link element_p3, mass 0.0001; visual cylinder length=0.0001 radius=0.01
Joints:
- removed joint joint_0_to_1
- added joint joint_0_to_p1: type continuous, parent element_first, child element_p1, origin xyz=0.0001 0 0 rpy=0 0.0 0, axis 0. 1. 0.
- added joint joint_p1_to_p2: type prismatic, parent element_p1, child element_p2, origin xyz=0.0001 0 0 rpy=0 0 0, axis 1. 0. 0., limit lower=-1.0 upper=0.0 effort=10000.0 velocity=10000.0
- added joint joint_p2_to_p3: type prismatic, parent element_p2, child element_p3, origin xyz=0.0001 0 0 rpy=0 0 0, axis 0. 1. 0., limit lower=-0.1 upper=0.1 effort=10000.0 velocity=10000.0
- added joint joint_p3_to_1: type prismatic, parent element_p3, child element_1, origin xyz=0.0001 0 0 rpy=0 0 0, axis 0. 0. 1., limit lower=-0.1 upper=0.1 effort=10000.0 velocity=10000.0

File: Tools/simulation/gz/models/cable_rod/model_orig.xacro (robot description, xacro)
@@ -74,41 +74,11 @@
     <xacro:tether_element elem_name="element_first" elem_length="${elem_length_ends}" elem_mass="${elem_mass_ends}" />
     <xacro:tether_element elem_name="element_last" elem_length="${elem_length_ends}" elem_mass="${elem_mass_ends}" />
-    <xacro:tether_element elem_name="element_p1" elem_length="${elem_length_ends}" elem_mass="${elem_mass_ends}" />
-    <xacro:tether_element elem_name="element_p2" elem_length="${elem_length_ends}" elem_mass="${elem_mass_ends}" />
-    <xacro:tether_element elem_name="element_p3" elem_length="${elem_length_ends}" elem_mass="${elem_mass_ends}" />
-    <!-- Load-side ball joint -->
-    <joint name="joint_0_to_p1" type="continuous">
+    <joint name="joint_0_to_1" type="continuous">
         <axis xyz="0. 1. 0."/>
         <origin xyz="${elem_length_ends} 0 0" rpy="0 ${ang_i/2} 0"/>
         <parent link="element_first"/>
-        <child link="element_p1"/>
+        <child link="element_1"/>
         <dynamics damping="${joint_damping}" friction="${joint_friction}"/>
     </joint>
-    <!-- Prismatic joints (controlling tension direction) -->
-    <joint name="joint_p1_to_p2" type="prismatic">
-        <origin xyz="${elem_length_ends} 0 0" rpy="0 0 0"/>
-        <parent link="element_p1"/>
-        <child link="element_p2"/>
-        <axis xyz="1. 0. 0."/>
-        <dynamics damping="0.0" friction="0.0"/>
-        <limit lower="-1.0" upper="0.0" effort="10000.0" velocity="10000.0"/>
-    </joint>
-    <joint name="joint_p2_to_p3" type="prismatic">
-        <origin xyz="${elem_length_ends} 0 0" rpy="0 0 0"/>
-        <parent link="element_p2"/>
-        <child link="element_p3"/>
-        <axis xyz="0. 1. 0."/>
-        <dynamics damping="0.0" friction="0.0"/>
-        <limit lower="-0.1" upper="0.1" effort="10000.0" velocity="10000.0"/>
-    </joint>
-    <joint name="joint_p3_to_1" type="prismatic">
-        <origin xyz="${elem_length_ends} 0 0" rpy="0 0 0"/>
-        <parent link="element_p3"/>
-        <child link="element_1"/>
-        <axis xyz="0. 0. 1."/>
-        <dynamics damping="0.0" friction="0.0"/>
-        <limit lower="-0.1" upper="0.1" effort="10000.0" velocity="10000.0"/>
-    </joint>
-    <!-- Drone-side ball joint -->
     <joint name="joint_${num_elements}_to_${num_elements+1}" type="continuous">
         <axis xyz="0. 1. 0."/>
