Commit message: Generated longer (~2m) cable

File: Tools/simulation/gz/models/tether/model.urdf (robot description, URDF)
Before this commit: robot tether, 12 links, 11 joints
Links:
- link element_1: geometry visual cylinder length=0.31286893008046185 radius=0.01
- link element_10: geometry visual cylinder length=0.31286893008046185 radius=0.01
- link element_2: geometry visual cylinder length=0.31286893008046185 radius=0.01
- link element_3: geometry visual cylinder length=0.31286893008046185 radius=0.01
- link element_4: geometry visual cylinder length=0.31286893008046185 radius=0.01
- link element_5: geometry visual cylinder length=0.31286893008046185 radius=0.01
- link element_6: geometry visual cylinder length=0.31286893008046185 radius=0.01
- link element_7: geometry visual cylinder length=0.31286893008046185 radius=0.01
- link element_8: geometry visual cylinder length=0.31286893008046185 radius=0.01
- link element_9: geometry visual cylinder length=0.31286893008046185 radius=0.01
Joints:
- joint joint_10_to_11: origin xyz=0.2190082510563233 0 0 rpy=0 1.413716694115407 0 -> xyz=0.31286893008046185 0 0 rpy=0 1.413716694115407 0
- joint joint_1_to_2: origin xyz=0.2190082510563233 0 0 rpy=0 -0.3141592653589793 0 -> xyz=0.31286893008046185 0 0 rpy=0 -0.3141592653589793 0
- joint joint_2_to_3: origin xyz=0.2190082510563233 0 0 rpy=0 -0.3141592653589793 0 -> xyz=0.31286893008046185 0 0 rpy=0 -0.3141592653589793 0
- joint joint_3_to_4: origin xyz=0.2190082510563233 0 0 rpy=0 -0.3141592653589793 0 -> xyz=0.31286893008046185 0 0 rpy=0 -0.3141592653589793 0
- joint joint_4_to_5: origin xyz=0.2190082510563233 0 0 rpy=0 -0.3141592653589793 0 -> xyz=0.31286893008046185 0 0 rpy=0 -0.3141592653589793 0
- joint joint_5_to_6: origin xyz=0.2190082510563233 0 0 rpy=0 -0.3141592653589793 0 -> xyz=0.31286893008046185 0 0 rpy=0 -0.3141592653589793 0
- joint joint_6_to_7: origin xyz=0.2190082510563233 0 0 rpy=0 -0.3141592653589793 0 -> xyz=0.31286893008046185 0 0 rpy=0 -0.3141592653589793 0
- joint joint_7_to_8: origin xyz=0.2190082510563233 0 0 rpy=0 -0.3141592653589793 0 -> xyz=0.31286893008046185 0 0 rpy=0 -0.3141592653589793 0
- joint joint_8_to_9: origin xyz=0.2190082510563233 0 0 rpy=0 -0.3141592653589793 0 -> xyz=0.31286893008046185 0 0 rpy=0 -0.3141592653589793 0
- joint joint_9_to_10: origin xyz=0.2190082510563233 0 0 rpy=0 -0.3141592653589793 0 -> xyz=0.31286893008046185 0 0 rpy=0 -0.3141592653589793 0

File: Tools/simulation/gz/models/tether/model_orig.xacro (robot description, xacro)
@@ -6,5 +6,5 @@
     These changes are now all defined in generate_sdf.sh-->
     <!-- Define properties -->
-    <xacro:property name="dist_connect_points" value="2.0" /> <!--1.4 - 1.42-->
+    <xacro:property name="dist_connect_points" value="1.4" /> <!--1.42-->
     <xacro:property name="tether_radius" value="0.01" />
     <xacro:property name="tether_mass" value="0.02" /> <!--0.1-->
