Commit message: Cable creation and drone moving fully automated with yaml file

File: Tools/simulation/gz/models/tether_2m/old/model.xacro (robot description, xacro)
@@ -1,37 +1,36 @@
 <?xml version="1.0" ?>
 <robot name="tether_2m" xmlns:xacro="http://ros.org/wiki/xacro">
-    <!-- Xacro to generate cable SDF -->
+    <!-- Xacro to generate tether SDF -->
     <!-- Note: need to manually find and replace all references to 'revolute'
-    with 'universal' in final SDF to get better cable. This also involves adding in a second axis.
+    with 'universal' in final SDF to get better tether. This also involves adding in a second axis.
     These changes are now all defined in generate_sdf.sh-->
     <!-- Define properties -->
     <!-- <xacro:property name="dist_connect_points" value="1.5475" />  -->
-    <xacro:property name="cable_radius" value="0.0031" />
-    <xacro:property name="cable_mass" value="0.02" />
-    <xacro:property name="cable_length" value="2.421" />
+    <xacro:property name="tether_radius" value="0.0031" />
+    <xacro:property name="tether_mass" value="0.02" />
+    <xacro:property name="tether_length" value="2.4210" />
     <xacro:property name="num_elements" value="10" />
     <xacro:property name="elem_length_ends" value="0.0001" />
+    <xacro:property name="elem_mass_main" value="${tether_mass/num_elements}" />
     <xacro:property name="elem_mass_ends" value="0.0001" />
-    <!-- Joint properties -->
     <xacro:property name="joint_friction" value="0" />
     <xacro:property name="joint_damping" value="0.01" />
     <!-- Calculations -->
-    <xacro:property name="elem_mass_main" value="${cable_mass/num_elements}" />
     <xacro:property name="ang_e" value="${pi/num_elements}"/>
     <xacro:property name="ang_i" value="${pi - ang_e}"/>
-    <xacro:property name="elem_length_main" value="${cable_length/num_elements}"/>
+    <xacro:property name="elem_length_main" value="${tether_length/num_elements}"/>
     <xacro:property name="dist_connect_points" value="${elem_length_main/sin(pi/(2*num_elements))}"/>
     <!-- Define link macro -->
-    <xacro:macro name="cable_element" params="elem_name elem_length elem_mass">
+    <xacro:macro name="tether_element" params="elem_name elem_length elem_mass">
         <link name="${elem_name}">
             <inertial>
                 <origin xyz="${elem_length/2} 0 0" rpy="0 ${pi/2} 0" />
                 <mass value="${elem_mass}"/>
-                <inertia ixx="${1/12*elem_mass*(3*cable_radius**2 + elem_length**2)}" ixy="0" ixz="0" iyy="${1/12*elem_mass*(3*cable_radius**2 + elem_length**2)}" iyz="0" izz="${1/2*elem_mass*(cable_radius**2)}" />
+                <inertia ixx="${1/12*elem_mass*(3*tether_radius**2 + elem_length**2)}" ixy="0" ixz="0" iyy="${1/12*elem_mass*(3*tether_radius**2 + elem_length**2)}" iyz="0" izz="${1/2*elem_mass*(tether_radius**2)}" />
             </inertial>
             <visual>
                 <origin xyz="${elem_length/2} 0 0" rpy="0 ${pi/2} 0" />
                 <geometry>
-                    <cylinder length="${elem_length}" radius="0.0031"/>
+                    <cylinder length="${elem_length}" radius="${tether_radius}"/>
                 </geometry>
             </visual>
@@ -39,5 +38,5 @@
                 <origin xyz="${elem_length/2} 0 0" rpy="0 ${pi/2} 0" />
                 <geometry>
-                    <cylinder length="${elem_length}" radius="0.0031"/> 0.0001
+                    <cylinder length="${elem_length}" radius="${tether_radius}"/> 0.0001
                 </geometry>
             </collision> -->
@@ -45,9 +44,9 @@
     </xacro:macro>
     <!-- Recursive loop to generate multiple elements and joints for said elements -->
-    <xacro:macro name="generate_cable" params="elem_num">
+    <xacro:macro name="generate_tether" params="elem_num">
         <!-- Generate elements and recurse-->
-        <xacro:cable_element elem_name="element_${elem_num}" elem_length="${elem_length_main}" elem_mass="${elem_mass_main}" />
+        <xacro:tether_element elem_name="element_${elem_num}" elem_length="${elem_length_main}" elem_mass="${elem_mass_main}" />
         <xacro:if value="${elem_num-1}">
-            <xacro:generate_cable elem_num="${elem_num-1}" />
+            <xacro:generate_tether elem_num="${elem_num-1}" />
         </xacro:if>
         <!-- Define joints -->
@@ -68,26 +67,26 @@
                 <parent link="element_${elem_num-1}"/>
                 <child link="element_${elem_num}"/>
-                <dynamics damping="0.01" friction="0"/>
+                <dynamics damping="${joint_damping}" friction="${joint_friction}"/>
             </joint>
         </xacro:if>
     </xacro:macro>
-    <!-- Call recursive loop to generate cable -->
-    <xacro:generate_cable elem_num="10" />
+    <!-- Call recursive loop to generate tether -->
+    <xacro:generate_tether elem_num="${num_elements}" />
     <!-- Add start and end elements and joints-->
-    <xacro:cable_element elem_name="element_first" elem_length="0.0001" elem_mass="0.0001" />
-    <xacro:cable_element elem_name="element_last" elem_length="0.0001" elem_mass="0.0001" />
+    <xacro:tether_element elem_name="element_first" elem_length="${elem_length_ends}" elem_mass="${elem_mass_ends}" />
+    <xacro:tether_element elem_name="element_last" elem_length="${elem_length_ends}" elem_mass="${elem_mass_ends}" />
     <joint name="joint_0_to_1" type="continuous">
         <axis xyz="0. 1. 0."/>
-        <origin xyz="0.0001 0 0" rpy="0 ${ang_i/2} 0"/>
+        <origin xyz="${elem_length_ends} 0 0" rpy="0 ${ang_i/2} 0"/>
         <parent link="element_first"/>
         <child link="element_1"/>
-        <dynamics damping="0.01" friction="0"/>
+        <dynamics damping="${joint_damping}" friction="${joint_friction}"/>
     </joint>
-    <joint name="joint_10_to_${num_elements+1}" type="continuous">
+    <joint name="joint_${num_elements}_to_${num_elements+1}" type="continuous">
         <axis xyz="0. 1. 0."/>
         <origin xyz="${elem_length_main} 0 0" rpy="0 ${(pi-ang_e)/2} 0"/>
-        <parent link="element_10"/>
+        <parent link="element_${num_elements}"/>
         <child link="element_last"/>
-        <dynamics damping="0.01" friction="0"/>
+        <dynamics damping="${joint_damping}" friction="${joint_friction}"/>
     </joint>
 </robot>

File: Tools/simulation/gz/models/tether_2m/template_model.xacro (robot description, xacro)
@@ -7,13 +7,13 @@
     <!-- Define properties -->
     <!-- <xacro:property name="dist_connect_points" value="1.5475" />  -->
-    <xacro:property name="cable_radius" value="0.0031" />
-    <xacro:property name="cable_mass" value="0.02" />
-    <xacro:property name="cable_length" value="2.421" />
-    <xacro:property name="num_elements" value="10" />
-    <xacro:property name="elem_length_ends" value="0.0001" />
-    <xacro:property name="elem_mass_ends" value="0.0001" />
+    <xacro:property name="cable_radius" value="${cable_radius}" />
+    <xacro:property name="cable_mass" value="${cable_mass}" />
+    <xacro:property name="cable_length" value="${cable_length}" />
+    <xacro:property name="num_elements" value="${num_elements}" />
+    <xacro:property name="elem_length_ends" value="${elem_length_ends}" />
+    <xacro:property name="elem_mass_ends" value="${elem_mass_ends}" />
     <!-- Joint properties -->
-    <xacro:property name="joint_friction" value="0" />
-    <xacro:property name="joint_damping" value="0.01" />
+    <xacro:property name="joint_friction" value="${joint_friction}" />
+    <xacro:property name="joint_damping" value="${joint_damping}" />
     <!-- Calculations -->
     <xacro:property name="elem_mass_main" value="${cable_mass/num_elements}" />
@@ -33,5 +33,5 @@
                 <origin xyz="${elem_length/2} 0 0" rpy="0 ${pi/2} 0" />
                 <geometry>
-                    <cylinder length="${elem_length}" radius="0.0031"/>
+                    <cylinder length="${elem_length}" radius="${cable_radius}"/>
                 </geometry>
             </visual>
@@ -39,5 +39,5 @@
                 <origin xyz="${elem_length/2} 0 0" rpy="0 ${pi/2} 0" />
                 <geometry>
-                    <cylinder length="${elem_length}" radius="0.0031"/> 0.0001
+                    <cylinder length="${elem_length}" radius="${cable_radius}"/> 0.0001
                 </geometry>
             </collision> -->
@@ -68,26 +68,26 @@
                 <parent link="element_${elem_num-1}"/>
                 <child link="element_${elem_num}"/>
-                <dynamics damping="0.01" friction="0"/>
+                <dynamics damping="${joint_damping}" friction="${joint_friction}"/>
             </joint>
         </xacro:if>
     </xacro:macro>
     <!-- Call recursive loop to generate cable -->
-    <xacro:generate_cable elem_num="10" />
+    <xacro:generate_cable elem_num="${num_elements}" />
     <!-- Add start and end elements and joints-->
-    <xacro:cable_element elem_name="element_first" elem_length="0.0001" elem_mass="0.0001" />
-    <xacro:cable_element elem_name="element_last" elem_length="0.0001" elem_mass="0.0001" />
+    <xacro:cable_element elem_name="element_first" elem_length="${elem_length_ends}" elem_mass="${elem_mass_ends}" />
+    <xacro:cable_element elem_name="element_last" elem_length="${elem_length_ends}" elem_mass="${elem_mass_ends}" />
     <joint name="joint_0_to_1" type="continuous">
         <axis xyz="0. 1. 0."/>
-        <origin xyz="0.0001 0 0" rpy="0 ${ang_i/2} 0"/>
+        <origin xyz="${elem_length_ends} 0 0" rpy="0 ${ang_i/2} 0"/>
         <parent link="element_first"/>
         <child link="element_1"/>
-        <dynamics damping="0.01" friction="0"/>
+        <dynamics damping="${joint_damping}" friction="${joint_friction}"/>
     </joint>
-    <joint name="joint_10_to_${num_elements+1}" type="continuous">
+    <joint name="joint_${num_elements}_to_${num_elements+1}" type="continuous">
         <axis xyz="0. 1. 0."/>
         <origin xyz="${elem_length_main} 0 0" rpy="0 ${(pi-ang_e)/2} 0"/>
-        <parent link="element_10"/>
+        <parent link="element_${num_elements}"/>
         <child link="element_last"/>
-        <dynamics damping="0.01" friction="0"/>
+        <dynamics damping="${joint_damping}" friction="${joint_friction}"/>
     </joint>
 </robot>
