Commit message: Updated tether to be correct length. Load has correct inertia

File: Tools/simulation/gz/models/tether_2m/model.urdf (robot description, URDF)
Before this commit: robot tether_2m, 12 links, 11 joints
Links:
- link element_1: geometry visual cylinder length=0.23793682132619123 radius=0.01
- link element_10: geometry visual cylinder length=0.23793682132619123 radius=0.01
- link element_2: geometry visual cylinder length=0.23793682132619123 radius=0.01
- link element_3: geometry visual cylinder length=0.23793682132619123 radius=0.01
- link element_4: geometry visual cylinder length=0.23793682132619123 radius=0.01
- link element_5: geometry visual cylinder length=0.23793682132619123 radius=0.01
- link element_6: geometry visual cylinder length=0.23793682132619123 radius=0.01
- link element_7: geometry visual cylinder length=0.23793682132619123 radius=0.01
- link element_8: geometry visual cylinder length=0.23793682132619123 radius=0.01
- link element_9: geometry visual cylinder length=0.23793682132619123 radius=0.01
Joints:
- joint joint_10_to_11: origin xyz=0.2190082510563233 0 0 rpy=0 1.413716694115407 0 -> xyz=0.23793682132619123 0 0 rpy=0 1.413716694115407 0
- joint joint_1_to_2: origin xyz=0.2190082510563233 0 0 rpy=0 -0.3141592653589793 0 -> xyz=0.23793682132619123 0 0 rpy=0 -0.3141592653589793 0
- joint joint_2_to_3: origin xyz=0.2190082510563233 0 0 rpy=0 -0.3141592653589793 0 -> xyz=0.23793682132619123 0 0 rpy=0 -0.3141592653589793 0
- joint joint_3_to_4: origin xyz=0.2190082510563233 0 0 rpy=0 -0.3141592653589793 0 -> xyz=0.23793682132619123 0 0 rpy=0 -0.3141592653589793 0
- joint joint_4_to_5: origin xyz=0.2190082510563233 0 0 rpy=0 -0.3141592653589793 0 -> xyz=0.23793682132619123 0 0 rpy=0 -0.3141592653589793 0
- joint joint_5_to_6: origin xyz=0.2190082510563233 0 0 rpy=0 -0.3141592653589793 0 -> xyz=0.23793682132619123 0 0 rpy=0 -0.3141592653589793 0
- joint joint_6_to_7: origin xyz=0.2190082510563233 0 0 rpy=0 -0.3141592653589793 0 -> xyz=0.23793682132619123 0 0 rpy=0 -0.3141592653589793 0
- joint joint_7_to_8: origin xyz=0.2190082510563233 0 0 rpy=0 -0.3141592653589793 0 -> xyz=0.23793682132619123 0 0 rpy=0 -0.3141592653589793 0
- joint joint_8_to_9: origin xyz=0.2190082510563233 0 0 rpy=0 -0.3141592653589793 0 -> xyz=0.23793682132619123 0 0 rpy=0 -0.3141592653589793 0
- joint joint_9_to_10: origin xyz=0.2190082510563233 0 0 rpy=0 -0.3141592653589793 0 -> xyz=0.23793682132619123 0 0 rpy=0 -0.3141592653589793 0

File: Tools/simulation/gz/models/tether_2m/model_pre_tune.xacro (robot description, xacro)
@@ -6,5 +6,5 @@
     These changes are now all defined in generate_sdf.sh-->
     <!-- Define properties -->
-    <xacro:property name="dist_connect_points" value="1.521" />
+    <xacro:property name="dist_connect_points" value="1.4" />
     <xacro:property name="tether_radius" value="0.01" />
     <xacro:property name="tether_mass" value="0.02" />
@@ -16,7 +16,7 @@
     <xacro:property name="joint_damping" value="0.01" />
     <!-- Calculations -->
+    <xacro:property name="elem_length_main" value="${(((dist_connect_points**2)/2)*(1-cos(ang_e)))**0.5}"/>
     <xacro:property name="ang_e" value="${pi/num_elements}"/>
     <xacro:property name="ang_i" value="${pi - ang_e}"/>
-    <xacro:property name="elem_length_main" value="${(((dist_connect_points**2)/2)*(1-cos(ang_e)))**0.5}"/>
     <!-- Define link macro -->
     <xacro:macro name="tether_element" params="elem_name elem_length elem_mass">

Commit message: Tuning cable length and load mass/inertia parameters

File: Tools/simulation/gz/models/tether_2m/model.urdf (robot description, URDF)
Before this commit: robot tether_2m, 12 links, 11 joints
Links:
- link element_1: geometry visual cylinder length=0.24169124848715678 radius=0.01
- link element_10: geometry visual cylinder length=0.24169124848715678 radius=0.01
- link element_2: geometry visual cylinder length=0.24169124848715678 radius=0.01
- link element_3: geometry visual cylinder length=0.24169124848715678 radius=0.01
- link element_4: geometry visual cylinder length=0.24169124848715678 radius=0.01
- link element_5: geometry visual cylinder length=0.24169124848715678 radius=0.01
- link element_6: geometry visual cylinder length=0.24169124848715678 radius=0.01
- link element_7: geometry visual cylinder length=0.24169124848715678 radius=0.01
- link element_8: geometry visual cylinder length=0.24169124848715678 radius=0.01
- link element_9: geometry visual cylinder length=0.24169124848715678 radius=0.01
Joints:
- joint joint_10_to_11: origin xyz=0.23793682132619123 0 0 rpy=0 1.413716694115407 0 -> xyz=0.24169124848715678 0 0 rpy=0 1.413716694115407 0
- joint joint_1_to_2: origin xyz=0.23793682132619123 0 0 rpy=0 -0.3141592653589793 0 -> xyz=0.24169124848715678 0 0 rpy=0 -0.3141592653589793 0
- joint joint_2_to_3: origin xyz=0.23793682132619123 0 0 rpy=0 -0.3141592653589793 0 -> xyz=0.24169124848715678 0 0 rpy=0 -0.3141592653589793 0
- joint joint_3_to_4: origin xyz=0.23793682132619123 0 0 rpy=0 -0.3141592653589793 0 -> xyz=0.24169124848715678 0 0 rpy=0 -0.3141592653589793 0
- joint joint_4_to_5: origin xyz=0.23793682132619123 0 0 rpy=0 -0.3141592653589793 0 -> xyz=0.24169124848715678 0 0 rpy=0 -0.3141592653589793 0
- joint joint_5_to_6: origin xyz=0.23793682132619123 0 0 rpy=0 -0.3141592653589793 0 -> xyz=0.24169124848715678 0 0 rpy=0 -0.3141592653589793 0
- joint joint_6_to_7: origin xyz=0.23793682132619123 0 0 rpy=0 -0.3141592653589793 0 -> xyz=0.24169124848715678 0 0 rpy=0 -0.3141592653589793 0
- joint joint_7_to_8: origin xyz=0.23793682132619123 0 0 rpy=0 -0.3141592653589793 0 -> xyz=0.24169124848715678 0 0 rpy=0 -0.3141592653589793 0
- joint joint_8_to_9: origin xyz=0.23793682132619123 0 0 rpy=0 -0.3141592653589793 0 -> xyz=0.24169124848715678 0 0 rpy=0 -0.3141592653589793 0
- joint joint_9_to_10: origin xyz=0.23793682132619123 0 0 rpy=0 -0.3141592653589793 0 -> xyz=0.24169124848715678 0 0 rpy=0 -0.3141592653589793 0

File: Tools/simulation/gz/models/tether_2m/model.xacro (robot description, xacro)
@@ -6,5 +6,5 @@
     These changes are now all defined in generate_sdf.sh-->
     <!-- Define properties -->
-    <xacro:property name="dist_connect_points" value="1.521" />
+    <xacro:property name="dist_connect_points" value="1.545" />
     <xacro:property name="tether_radius" value="0.01" />
     <xacro:property name="tether_mass" value="0.02" />

File: Tools/simulation/gz/models/tether_2m/model_2.38.xacro (robot description, xacro)
@@ -6,5 +6,5 @@
     These changes are now all defined in generate_sdf.sh-->
     <!-- Define properties -->
-    <xacro:property name="dist_connect_points" value="1.4" />
+    <xacro:property name="dist_connect_points" value="1.521" />
     <xacro:property name="tether_radius" value="0.01" />
     <xacro:property name="tether_mass" value="0.02" />
@@ -16,7 +16,7 @@
     <xacro:property name="joint_damping" value="0.01" />
     <!-- Calculations -->
-    <xacro:property name="elem_length_main" value="${(((dist_connect_points**2)/2)*(1-cos(ang_e)))**0.5}"/>
     <xacro:property name="ang_e" value="${pi/num_elements}"/>
     <xacro:property name="ang_i" value="${pi - ang_e}"/>
+    <xacro:property name="elem_length_main" value="${(((dist_connect_points**2)/2)*(1-cos(ang_e)))**0.5}"/>
     <!-- Define link macro -->
     <xacro:macro name="tether_element" params="elem_name elem_length elem_mass">

Commit message: Basic tether of correct length and radius complete. Before parameter sensitivity study

File: Tools/simulation/gz/models/tether_2m/model.urdf (robot description, URDF)
Before this commit: robot tether_2m, 12 links, 11 joints
Links:
- link element_1: geometry visual cylinder length=0.24209999999999998 radius=0.0031
- link element_10: geometry visual cylinder length=0.24209999999999998 radius=0.0031
- link element_2: geometry visual cylinder length=0.24209999999999998 radius=0.0031
- link element_3: geometry visual cylinder length=0.24209999999999998 radius=0.0031
- link element_4: geometry visual cylinder length=0.24209999999999998 radius=0.0031
- link element_5: geometry visual cylinder length=0.24209999999999998 radius=0.0031
- link element_6: geometry visual cylinder length=0.24209999999999998 radius=0.0031
- link element_7: geometry visual cylinder length=0.24209999999999998 radius=0.0031
- link element_8: geometry visual cylinder length=0.24209999999999998 radius=0.0031
- link element_9: geometry visual cylinder length=0.24209999999999998 radius=0.0031
- link element_first: geometry visual cylinder length=0.0001 radius=0.0031
- link element_last: geometry visual cylinder length=0.0001 radius=0.0031
Joints:
- joint joint_10_to_11: origin xyz=0.24169124848715678 0 0 rpy=0 1.413716694115407 0 -> xyz=0.24209999999999998 0 0 rpy=0 1.413716694115407 0
- joint joint_1_to_2: origin xyz=0.24169124848715678 0 0 rpy=0 -0.3141592653589793 0 -> xyz=0.24209999999999998 0 0 rpy=0 -0.3141592653589793 0
- joint joint_2_to_3: origin xyz=0.24169124848715678 0 0 rpy=0 -0.3141592653589793 0 -> xyz=0.24209999999999998 0 0 rpy=0 -0.3141592653589793 0
- joint joint_3_to_4: origin xyz=0.24169124848715678 0 0 rpy=0 -0.3141592653589793 0 -> xyz=0.24209999999999998 0 0 rpy=0 -0.3141592653589793 0
- joint joint_4_to_5: origin xyz=0.24169124848715678 0 0 rpy=0 -0.3141592653589793 0 -> xyz=0.24209999999999998 0 0 rpy=0 -0.3141592653589793 0
- joint joint_5_to_6: origin xyz=0.24169124848715678 0 0 rpy=0 -0.3141592653589793 0 -> xyz=0.24209999999999998 0 0 rpy=0 -0.3141592653589793 0
- joint joint_6_to_7: origin xyz=0.24169124848715678 0 0 rpy=0 -0.3141592653589793 0 -> xyz=0.24209999999999998 0 0 rpy=0 -0.3141592653589793 0
- joint joint_7_to_8: origin xyz=0.24169124848715678 0 0 rpy=0 -0.3141592653589793 0 -> xyz=0.24209999999999998 0 0 rpy=0 -0.3141592653589793 0
- joint joint_8_to_9: origin xyz=0.24169124848715678 0 0 rpy=0 -0.3141592653589793 0 -> xyz=0.24209999999999998 0 0 rpy=0 -0.3141592653589793 0
- joint joint_9_to_10: origin xyz=0.24169124848715678 0 0 rpy=0 -0.3141592653589793 0 -> xyz=0.24209999999999998 0 0 rpy=0 -0.3141592653589793 0

File: Tools/simulation/gz/models/tether_2m/model_old.xacro (robot description, xacro)
@@ -6,8 +6,7 @@
     These changes are now all defined in generate_sdf.sh-->
     <!-- Define properties -->
-    <!-- <xacro:property name="dist_connect_points" value="1.5475" />  -->
+    <xacro:property name="dist_connect_points" value="1.5475" />
     <xacro:property name="tether_radius" value="0.0031" />
     <xacro:property name="tether_mass" value="0.02" />
-    <xacro:property name="tether_length" value="2.4210" />
     <xacro:property name="num_elements" value="10" />
     <xacro:property name="elem_length_ends" value="0.0001" />
@@ -19,6 +18,5 @@
     <xacro:property name="ang_e" value="${pi/num_elements}"/>
     <xacro:property name="ang_i" value="${pi - ang_e}"/>
-    <xacro:property name="elem_length_main" value="${tether_length/num_elements}"/>
-    <xacro:property name="dist_connect_points" value="${elem_length_main/sin(pi/(2*num_elements))}"/>
+    <xacro:property name="elem_length_main" value="${(((dist_connect_points**2)/2)*(1-cos(ang_e)))**0.5}"/>
     <!-- Define link macro -->
     <xacro:macro name="tether_element" params="elem_name elem_length elem_mass">
