Commit message: Generating straight tether in progress

File: Tools/simulation/gz/models/tether_2m/model.urdf (robot description, URDF)
Before this commit: robot tether_2m, 12 links, 11 joints
Joints:
- joint joint_0_to_1: axis 0. 1. 0. -> 0 1 0; origin xyz=0.0001 0 0 rpy=0 1.413716694115407 0 -> xyz=0 0 0.0001 rpy=0 0 0
- joint joint_10_to_11: axis 0. 1. 0. -> 0 1 0; origin xyz=0.24209999999999998 0 0 rpy=0 1.413716694115407 0 -> xyz=0 0 0.24209999999999998 rpy=0 0 0
- joint joint_1_to_2: axis 0. 1. 0. -> 0 1 0; origin xyz=0.24209999999999998 0 0 rpy=0 -0.3141592653589793 0 -> xyz=0 0 0.24209999999999998 rpy=0 0 0
- joint joint_2_to_3: axis 0. 1. 0. -> 0 1 0; origin xyz=0.24209999999999998 0 0 rpy=0 -0.3141592653589793 0 -> xyz=0 0 0.24209999999999998 rpy=0 0 0
- joint joint_3_to_4: axis 0. 1. 0. -> 0 1 0; origin xyz=0.24209999999999998 0 0 rpy=0 -0.3141592653589793 0 -> xyz=0 0 0.24209999999999998 rpy=0 0 0
- joint joint_4_to_5: axis 0. 1. 0. -> 0 1 0; origin xyz=0.24209999999999998 0 0 rpy=0 -0.3141592653589793 0 -> xyz=0 0 0.24209999999999998 rpy=0 0 0
- joint joint_5_to_6: axis 0. 1. 0. -> 0 1 0; origin xyz=0.24209999999999998 0 0 rpy=0 -0.3141592653589793 0 -> xyz=0 0 0.24209999999999998 rpy=0 0 0
- joint joint_6_to_7: axis 0. 1. 0. -> 0 1 0; origin xyz=0.24209999999999998 0 0 rpy=0 -0.3141592653589793 0 -> xyz=0 0 0.24209999999999998 rpy=0 0 0
- joint joint_7_to_8: axis 0. 1. 0. -> 0 1 0; origin xyz=0.24209999999999998 0 0 rpy=0 -0.3141592653589793 0 -> xyz=0 0 0.24209999999999998 rpy=0 0 0
- joint joint_8_to_9: axis 0. 1. 0. -> 0 1 0; origin xyz=0.24209999999999998 0 0 rpy=0 -0.3141592653589793 0 -> xyz=0 0 0.24209999999999998 rpy=0 0 0
- joint joint_9_to_10: axis 0. 1. 0. -> 0 1 0; origin xyz=0.24209999999999998 0 0 rpy=0 -0.3141592653589793 0 -> xyz=0 0 0.24209999999999998 rpy=0 0 0

File: Tools/simulation/gz/models/tether_2m/model.xacro (robot description, xacro)
@@ -1,93 +1,98 @@
 <?xml version="1.0" ?>
 <robot name="tether_2m" xmlns:xacro="http://ros.org/wiki/xacro">
-    <!-- Xacro to generate cable SDF -->
-    <!-- Note: need to manually find and replace all references to 'revolute'
-    with 'universal' in final SDF to get better cable. This also involves adding in a second axis.
-    These changes are now all defined in generate_sdf.sh-->
-    <!-- Define properties -->
-    <!-- <xacro:property name="dist_connect_points" value="1.5475" />  -->
-    <xacro:property name="cable_radius" value="0.0031" />
-    <xacro:property name="cable_mass" value="0.02" />
-    <xacro:property name="cable_length" value="2.421" />
-    <xacro:property name="num_elements" value="10" />
-    <xacro:property name="elem_length_ends" value="0.0001" />
-    <xacro:property name="elem_mass_ends" value="0.0001" />
-    <!-- Joint properties -->
-    <xacro:property name="joint_friction" value="0" />
-    <xacro:property name="joint_damping" value="0.01" />
-    <!-- Calculations -->
-    <xacro:property name="elem_mass_main" value="${cable_mass/num_elements}" />
-    <xacro:property name="ang_e" value="${pi/num_elements}"/>
-    <xacro:property name="ang_i" value="${pi - ang_e}"/>
-    <xacro:property name="elem_length_main" value="${cable_length/num_elements}"/>
-    <xacro:property name="dist_connect_points" value="${elem_length_main/sin(pi/(2*num_elements))}"/>
-    <!-- Define link macro -->
-    <xacro:macro name="cable_element" params="elem_name elem_length elem_mass">
-        <link name="${elem_name}">
-            <inertial>
-                <origin xyz="${elem_length/2} 0 0" rpy="0 ${pi/2} 0" />
-                <mass value="${elem_mass}"/>
-                <inertia ixx="${1/12*elem_mass*(3*cable_radius**2 + elem_length**2)}" ixy="0" ixz="0" iyy="${1/12*elem_mass*(3*cable_radius**2 + elem_length**2)}" iyz="0" izz="${1/2*elem_mass*(cable_radius**2)}" />
-            </inertial>
-            <visual>
-                <origin xyz="${elem_length/2} 0 0" rpy="0 ${pi/2} 0" />
-                <geometry>
-                    <cylinder length="${elem_length}" radius="0.0031"/>
-                </geometry>
-            </visual>
-            <!-- <collision>
-                <origin xyz="${elem_length/2} 0 0" rpy="0 ${pi/2} 0" />
-                <geometry>
-                    <cylinder length="${elem_length}" radius="0.0031"/> 0.0001
-                </geometry>
-            </collision> -->
-        </link>
-    </xacro:macro>
-    <!-- Recursive loop to generate multiple elements and joints for said elements -->
-    <xacro:macro name="generate_cable" params="elem_num">
-        <!-- Generate elements and recurse-->
-        <xacro:cable_element elem_name="element_${elem_num}" elem_length="${elem_length_main}" elem_mass="${elem_mass_main}" />
-        <xacro:if value="${elem_num-1}">
-            <xacro:generate_cable elem_num="${elem_num-1}" />
-        </xacro:if>
-        <!-- Define joints -->
-        <xacro:if value="${elem_num-1 > 0}">
-            <joint name="joint_${elem_num-1}_to_${elem_num}" type="continuous">
-                <axis xyz="0. 1. 0."/>
-                <!-- <axis xyz="0. 1. 1."/> -->
-                <origin xyz="${elem_length_main} 0 0" rpy="0 ${-ang_e} 0"/>
-                <!-- <xacro:if value="${elem_num  == 1}">
-                    <origin xyz="${elem_length_main} 0 0" rpy="0 ${ang_i/2} 0"/>
-                </xacro:if>
-                <xacro:if value="${elem_num  == num_elements}">
-                    <origin xyz="${elem_length_main} 0 0" rpy="0 ${(pi-ang_e)/2} 0"/>
-                </xacro:if>
-                <xacro:if value="${(elem_num > 1) and (elem_num < num_elements)}">
-                    <origin xyz="${elem_length_main} 0 0" rpy="0 ${-ang_e} 0"/>
-                </xacro:if> -->
-                <parent link="element_${elem_num-1}"/>
-                <child link="element_${elem_num}"/>
-                <dynamics damping="0.01" friction="0"/>
-            </joint>
-        </xacro:if>
-    </xacro:macro>
-    <!-- Call recursive loop to generate cable -->
-    <xacro:generate_cable elem_num="10" />
-    <!-- Add start and end elements and joints-->
-    <xacro:cable_element elem_name="element_first" elem_length="0.0001" elem_mass="0.0001" />
-    <xacro:cable_element elem_name="element_last" elem_length="0.0001" elem_mass="0.0001" />
-    <joint name="joint_0_to_1" type="continuous">
-        <axis xyz="0. 1. 0."/>
-        <origin xyz="0.0001 0 0" rpy="0 ${ang_i/2} 0"/>
-        <parent link="element_first"/>
-        <child link="element_1"/>
-        <dynamics damping="0.01" friction="0"/>
-    </joint>
-    <joint name="joint_10_to_${num_elements+1}" type="continuous">
-        <axis xyz="0. 1. 0."/>
-        <origin xyz="${elem_length_main} 0 0" rpy="0 ${(pi-ang_e)/2} 0"/>
-        <parent link="element_10"/>
-        <child link="element_last"/>
-        <dynamics damping="0.01" friction="0"/>
-    </joint>
+  <!-- Properties -->
+  <xacro:property name="cable_radius"     value="0.0031" />
+  <xacro:property name="cable_mass"       value="0.02" />
+  <xacro:property name="cable_length"     value="2.421" />
+  <xacro:property name="num_elements"     value="10" />
+  <xacro:property name="elem_length_ends" value="0.0001" />
+  <xacro:property name="elem_mass_ends"   value="0.0001" />
+  <!-- Joint properties -->
+  <xacro:property name="joint_friction" value="5" />
+  <xacro:property name="joint_damping"  value="0.01"  />
+  <!-- <xacro:property name="joint_effort"   value="1000" />
+  <xacro:property name="joint_velocity" value="1000" /> -->
+  <!-- Derived values -->
+  <xacro:property name="elem_mass_main"   value="${cable_mass/num_elements}" />
+  <xacro:property name="elem_length_main" value="${cable_length/num_elements}" />
+  <!-- Legacy placeholders kept for template compatibility -->
+  <xacro:property name="ang_e" value="${pi/num_elements}"/>
+  <xacro:property name="ang_i" value="${pi - ang_e}"/>
+  <xacro:property name="dist_connect_points" value="${elem_length_main/sin(pi/(2*num_elements))}"/>
+  <!-- Link macro -->
+  <xacro:macro name="cable_element" params="elem_name elem_length elem_mass">
+    <link name="${elem_name}">
+      <inertial>
+        <origin xyz="0 0 ${elem_length/2}" rpy="0 0 0"/>
+        <mass value="${elem_mass}"/>
+        <inertia
+          ixx="${(1.0/12.0)*elem_mass*(3*cable_radius*cable_radius + elem_length*elem_length)}"
+          ixy="0" ixz="0"
+          iyy="${(1.0/12.0)*elem_mass*(3*cable_radius*cable_radius + elem_length*elem_length)}"
+          iyz="0"
+          izz="${0.5*elem_mass*(cable_radius*cable_radius)}"/>
+      </inertial>
+      <visual>
+        <origin xyz="0 0 ${elem_length/2}" rpy="0 0 0"/>
+        <geometry>
+          <cylinder length="${elem_length}" radius="0.0031"/>
+        </geometry>
+      </visual>
+      <!-- <collision>
+        <origin xyz="0 0 ${elem_length/2}" rpy="0 0 0"/>
+        <geometry>
+          <cylinder length="${elem_length}" radius="0.0031"/>
+        </geometry>
+      </collision> -->
+    </link>
+  </xacro:macro>
+  <!-- Recursive chain -->
+  <xacro:macro name="generate_cable" params="elem_num">
+    <xacro:cable_element elem_name="element_${elem_num}"
+                         elem_length="${elem_length_main}"
+                         elem_mass="${elem_mass_main}"/>
+    <xacro:if value="${elem_num-1}">
+      <xacro:generate_cable elem_num="${elem_num-1}" />
+    </xacro:if>
+    <xacro:if value="${elem_num-1 > 0}">
+      <joint name="joint_${elem_num-1}_to_${elem_num}" type="continuous">
+        <axis xyz="0 1 0">
+          <!-- <limit effort="${joint_effort}" velocity="${joint_velocity}"/> -->
+          <dynamics damping="0.01" friction="5"/>
+        </axis>
+        <origin xyz="0 0 ${elem_length_main}" rpy="0 0 0"/>
+        <parent link="element_${elem_num-1}"/>
+        <child  link="element_${elem_num}"/>
+      </joint>
+    </xacro:if>
+  </xacro:macro>
+  <!-- Interior chain -->
+  <xacro:generate_cable elem_num="10" />
+  <!-- Endcaps -->
+  <xacro:cable_element elem_name="element_first"
+                       elem_length="0.0001"
+                       elem_mass="0.0001"/>
+  <xacro:cable_element elem_name="element_last"
+                       elem_length="0.0001"
+                       elem_mass="0.0001"/>
+  <!-- First to element_1 -->
+  <joint name="joint_0_to_1" type="continuous">
+    <axis xyz="0 1 0">
+      <!-- <limit effort="${joint_effort}" velocity="${joint_velocity}"/> -->
+      <dynamics damping="0.01" friction="5"/>
+    </axis>
+    <origin xyz="0 0 0.0001" rpy="0 0 0"/>
+    <parent link="element_first"/>
+    <child  link="element_1"/>
+  </joint>
+  <!-- Last interior to endcap -->
+  <joint name="joint_10_to_${num_elements+1}" type="continuous">
+    <axis xyz="0 1 0">
+      <!-- <limit effort="${joint_effort}" velocity="${joint_velocity}"/> -->
+      <dynamics damping="0.01" friction="5"/>
+    </axis>
+    <origin xyz="0 0 ${elem_length_main}" rpy="0 0 0"/>
+    <parent link="element_10"/>
+    <child  link="element_last"/>
+  </joint>
 </robot>

File: Tools/simulation/gz/models/tether_2m/template_model.xacro (robot description, xacro)
@@ -1,93 +1,98 @@
 <?xml version="1.0" ?>
 <robot name="tether_2m" xmlns:xacro="http://ros.org/wiki/xacro">
-    <!-- Xacro to generate cable SDF -->
-    <!-- Note: need to manually find and replace all references to 'revolute'
-    with 'universal' in final SDF to get better cable. This also involves adding in a second axis.
-    These changes are now all defined in generate_sdf.sh-->
-    <!-- Define properties -->
-    <!-- <xacro:property name="dist_connect_points" value="1.5475" />  -->
-    <xacro:property name="cable_radius" value="${cable_radius}" />
-    <xacro:property name="cable_mass" value="${cable_mass}" />
-    <xacro:property name="cable_length" value="${cable_length}" />
-    <xacro:property name="num_elements" value="${num_elements}" />
-    <xacro:property name="elem_length_ends" value="${elem_length_ends}" />
-    <xacro:property name="elem_mass_ends" value="${elem_mass_ends}" />
-    <!-- Joint properties -->
-    <xacro:property name="joint_friction" value="${joint_friction}" />
-    <xacro:property name="joint_damping" value="${joint_damping}" />
-    <!-- Calculations -->
-    <xacro:property name="elem_mass_main" value="${cable_mass/num_elements}" />
-    <xacro:property name="ang_e" value="${pi/num_elements}"/>
-    <xacro:property name="ang_i" value="${pi - ang_e}"/>
-    <xacro:property name="elem_length_main" value="${cable_length/num_elements}"/>
-    <xacro:property name="dist_connect_points" value="${elem_length_main/sin(pi/(2*num_elements))}"/>
-    <!-- Define link macro -->
-    <xacro:macro name="cable_element" params="elem_name elem_length elem_mass">
-        <link name="${elem_name}">
-            <inertial>
-                <origin xyz="${elem_length/2} 0 0" rpy="0 ${pi/2} 0" />
-                <mass value="${elem_mass}"/>
-                <inertia ixx="${1/12*elem_mass*(3*cable_radius**2 + elem_length**2)}" ixy="0" ixz="0" iyy="${1/12*elem_mass*(3*cable_radius**2 + elem_length**2)}" iyz="0" izz="${1/2*elem_mass*(cable_radius**2)}" />
-            </inertial>
-            <visual>
-                <origin xyz="${elem_length/2} 0 0" rpy="0 ${pi/2} 0" />
-                <geometry>
-                    <cylinder length="${elem_length}" radius="${cable_radius}"/>
-                </geometry>
-            </visual>
-            <!-- <collision>
-                <origin xyz="${elem_length/2} 0 0" rpy="0 ${pi/2} 0" />
-                <geometry>
-                    <cylinder length="${elem_length}" radius="${cable_radius}"/> 0.0001
-                </geometry>
-            </collision> -->
-        </link>
-    </xacro:macro>
-    <!-- Recursive loop to generate multiple elements and joints for said elements -->
-    <xacro:macro name="generate_cable" params="elem_num">
-        <!-- Generate elements and recurse-->
-        <xacro:cable_element elem_name="element_${elem_num}" elem_length="${elem_length_main}" elem_mass="${elem_mass_main}" />
-        <xacro:if value="${elem_num-1}">
-            <xacro:generate_cable elem_num="${elem_num-1}" />
-        </xacro:if>
-        <!-- Define joints -->
-        <xacro:if value="${elem_num-1 > 0}">
-            <joint name="joint_${elem_num-1}_to_${elem_num}" type="continuous">
-                <axis xyz="0. 1. 0."/>
-                <!-- <axis xyz="0. 1. 1."/> -->
-                <origin xyz="${elem_length_main} 0 0" rpy="0 ${-ang_e} 0"/>
-                <!-- <xacro:if value="${elem_num  == 1}">
-                    <origin xyz="${elem_length_main} 0 0" rpy="0 ${ang_i/2} 0"/>
-                </xacro:if>
-                <xacro:if value="${elem_num  == num_elements}">
-                    <origin xyz="${elem_length_main} 0 0" rpy="0 ${(pi-ang_e)/2} 0"/>
-                </xacro:if>
-                <xacro:if value="${(elem_num > 1) and (elem_num < num_elements)}">
-                    <origin xyz="${elem_length_main} 0 0" rpy="0 ${-ang_e} 0"/>
-                </xacro:if> -->
-                <parent link="element_${elem_num-1}"/>
-                <child link="element_${elem_num}"/>
-                <dynamics damping="${joint_damping}" friction="${joint_friction}"/>
-            </joint>
-        </xacro:if>
-    </xacro:macro>
-    <!-- Call recursive loop to generate cable -->
-    <xacro:generate_cable elem_num="${num_elements}" />
-    <!-- Add start and end elements and joints-->
-    <xacro:cable_element elem_name="element_first" elem_length="${elem_length_ends}" elem_mass="${elem_mass_ends}" />
-    <xacro:cable_element elem_name="element_last" elem_length="${elem_length_ends}" elem_mass="${elem_mass_ends}" />
-    <joint name="joint_0_to_1" type="continuous">
-        <axis xyz="0. 1. 0."/>
-        <origin xyz="${elem_length_ends} 0 0" rpy="0 ${ang_i/2} 0"/>
-        <parent link="element_first"/>
-        <child link="element_1"/>
-        <dynamics damping="${joint_damping}" friction="${joint_friction}"/>
-    </joint>
-    <joint name="joint_${num_elements}_to_${num_elements+1}" type="continuous">
-        <axis xyz="0. 1. 0."/>
-        <origin xyz="${elem_length_main} 0 0" rpy="0 ${(pi-ang_e)/2} 0"/>
-        <parent link="element_${num_elements}"/>
-        <child link="element_last"/>
-        <dynamics damping="${joint_damping}" friction="${joint_friction}"/>
-    </joint>
+  <!-- Properties -->
+  <xacro:property name="cable_radius"     value="${cable_radius}" />
+  <xacro:property name="cable_mass"       value="${cable_mass}" />
+  <xacro:property name="cable_length"     value="${cable_length}" />
+  <xacro:property name="num_elements"     value="${num_elements}" />
+  <xacro:property name="elem_length_ends" value="${elem_length_ends}" />
+  <xacro:property name="elem_mass_ends"   value="${elem_mass_ends}" />
+  <!-- Joint properties -->
+  <xacro:property name="joint_friction" value="${joint_friction}" />
+  <xacro:property name="joint_damping"  value="${joint_damping}"  />
+  <!-- <xacro:property name="joint_effort"   value="1000" />
+  <xacro:property name="joint_velocity" value="1000" /> -->
+  <!-- Derived values -->
+  <xacro:property name="elem_mass_main"   value="${cable_mass/num_elements}" />
+  <xacro:property name="elem_length_main" value="${cable_length/num_elements}" />
+  <!-- Legacy placeholders kept for template compatibility -->
+  <xacro:property name="ang_e" value="${pi/num_elements}"/>
+  <xacro:property name="ang_i" value="${pi - ang_e}"/>
+  <xacro:property name="dist_connect_points" value="${elem_length_main/sin(pi/(2*num_elements))}"/>
+  <!-- Link macro -->
+  <xacro:macro name="cable_element" params="elem_name elem_length elem_mass">
+    <link name="${elem_name}">
+      <inertial>
+        <origin xyz="0 0 ${elem_length/2}" rpy="0 0 0"/>
+        <mass value="${elem_mass}"/>
+        <inertia
+          ixx="${(1.0/12.0)*elem_mass*(3*cable_radius*cable_radius + elem_length*elem_length)}"
+          ixy="0" ixz="0"
+          iyy="${(1.0/12.0)*elem_mass*(3*cable_radius*cable_radius + elem_length*elem_length)}"
+          iyz="0"
+          izz="${0.5*elem_mass*(cable_radius*cable_radius)}"/>
+      </inertial>
+      <visual>
+        <origin xyz="0 0 ${elem_length/2}" rpy="0 0 0"/>
+        <geometry>
+          <cylinder length="${elem_length}" radius="${cable_radius}"/>
+        </geometry>
+      </visual>
+      <!-- <collision>
+        <origin xyz="0 0 ${elem_length/2}" rpy="0 0 0"/>
+        <geometry>
+          <cylinder length="${elem_length}" radius="${cable_radius}"/>
+        </geometry>
+      </collision> -->
+    </link>
+  </xacro:macro>
+  <!-- Recursive chain -->
+  <xacro:macro name="generate_cable" params="elem_num">
+    <xacro:cable_element elem_name="element_${elem_num}"
+                         elem_length="${elem_length_main}"
+                         elem_mass="${elem_mass_main}"/>
+    <xacro:if value="${elem_num-1}">
+      <xacro:generate_cable elem_num="${elem_num-1}" />
+    </xacro:if>
+    <xacro:if value="${elem_num-1 > 0}">
+      <joint name="joint_${elem_num-1}_to_${elem_num}" type="continuous">
+        <axis xyz="0 1 0">
+          <!-- <limit effort="${joint_effort}" velocity="${joint_velocity}"/> -->
+          <dynamics damping="${joint_damping}" friction="${joint_friction}"/>
+        </axis>
+        <origin xyz="0 0 ${elem_length_main}" rpy="0 0 0"/>
+        <parent link="element_${elem_num-1}"/>
+        <child  link="element_${elem_num}"/>
+      </joint>
+    </xacro:if>
+  </xacro:macro>
+  <!-- Interior chain -->
+  <xacro:generate_cable elem_num="${num_elements}" />
+  <!-- Endcaps -->
+  <xacro:cable_element elem_name="element_first"
+                       elem_length="${elem_length_ends}"
+                       elem_mass="${elem_mass_ends}"/>
+  <xacro:cable_element elem_name="element_last"
+                       elem_length="${elem_length_ends}"
+                       elem_mass="${elem_mass_ends}"/>
+  <!-- First to element_1 -->
+  <joint name="joint_0_to_1" type="continuous">
+    <axis xyz="0 1 0">
+      <!-- <limit effort="${joint_effort}" velocity="${joint_velocity}"/> -->
+      <dynamics damping="${joint_damping}" friction="${joint_friction}"/>
+    </axis>
+    <origin xyz="0 0 ${elem_length_ends}" rpy="0 0 0"/>
+    <parent link="element_first"/>
+    <child  link="element_1"/>
+  </joint>
+  <!-- Last interior to endcap -->
+  <joint name="joint_${num_elements}_to_${num_elements+1}" type="continuous">
+    <axis xyz="0 1 0">
+      <!-- <limit effort="${joint_effort}" velocity="${joint_velocity}"/> -->
+      <dynamics damping="${joint_damping}" friction="${joint_friction}"/>
+    </axis>
+    <origin xyz="0 0 ${elem_length_main}" rpy="0 0 0"/>
+    <parent link="element_${num_elements}"/>
+    <child  link="element_last"/>
+  </joint>
 </robot>
