Commit message: Can generate cable with alternating joints. Bent cable is best (straight still exists if needed)

File: Tools/simulation/gz/models/tether_2m/template_model.xacro (robot description, xacro)
@@ -1,98 +1,93 @@
 <?xml version="1.0" ?>
 <robot name="tether_2m" xmlns:xacro="http://ros.org/wiki/xacro">
-  <!-- Properties -->
-  <xacro:property name="cable_radius"     value="${cable_radius}" />
-  <xacro:property name="cable_mass"       value="${cable_mass}" />
-  <xacro:property name="cable_length"     value="${cable_length}" />
-  <xacro:property name="num_elements"     value="${num_elements}" />
-  <xacro:property name="elem_length_ends" value="${elem_length_ends}" />
-  <xacro:property name="elem_mass_ends"   value="${elem_mass_ends}" />
-  <!-- Joint properties -->
-  <xacro:property name="joint_friction" value="${joint_friction}" />
-  <xacro:property name="joint_damping"  value="${joint_damping}"  />
-  <!-- <xacro:property name="joint_effort"   value="1000" />
-  <xacro:property name="joint_velocity" value="1000" /> -->
-  <!-- Derived values -->
-  <xacro:property name="elem_mass_main"   value="${cable_mass/num_elements}" />
-  <xacro:property name="elem_length_main" value="${cable_length/num_elements}" />
-  <!-- Legacy placeholders kept for template compatibility -->
-  <xacro:property name="ang_e" value="${pi/num_elements}"/>
-  <xacro:property name="ang_i" value="${pi - ang_e}"/>
-  <xacro:property name="dist_connect_points" value="${elem_length_main/sin(pi/(2*num_elements))}"/>
-  <!-- Link macro -->
-  <xacro:macro name="cable_element" params="elem_name elem_length elem_mass">
-    <link name="${elem_name}">
-      <inertial>
-        <origin xyz="0 0 ${elem_length/2}" rpy="0 0 0"/>
-        <mass value="${elem_mass}"/>
-        <inertia
-          ixx="${(1.0/12.0)*elem_mass*(3*cable_radius*cable_radius + elem_length*elem_length)}"
-          ixy="0" ixz="0"
-          iyy="${(1.0/12.0)*elem_mass*(3*cable_radius*cable_radius + elem_length*elem_length)}"
-          iyz="0"
-          izz="${0.5*elem_mass*(cable_radius*cable_radius)}"/>
-      </inertial>
-      <visual>
-        <origin xyz="0 0 ${elem_length/2}" rpy="0 0 0"/>
-        <geometry>
-          <cylinder length="${elem_length}" radius="${cable_radius}"/>
-        </geometry>
-      </visual>
-      <!-- <collision>
-        <origin xyz="0 0 ${elem_length/2}" rpy="0 0 0"/>
-        <geometry>
-          <cylinder length="${elem_length}" radius="${cable_radius}"/>
-        </geometry>
-      </collision> -->
-    </link>
-  </xacro:macro>
-  <!-- Recursive chain -->
-  <xacro:macro name="generate_cable" params="elem_num">
-    <xacro:cable_element elem_name="element_${elem_num}"
-                         elem_length="${elem_length_main}"
-                         elem_mass="${elem_mass_main}"/>
-    <xacro:if value="${elem_num-1}">
-      <xacro:generate_cable elem_num="${elem_num-1}" />
-    </xacro:if>
-    <xacro:if value="${elem_num-1 > 0}">
-      <joint name="joint_${elem_num-1}_to_${elem_num}" type="continuous">
-        <axis xyz="0 1 0">
-          <!-- <limit effort="${joint_effort}" velocity="${joint_velocity}"/> -->
-          <dynamics damping="${joint_damping}" friction="${joint_friction}"/>
-        </axis>
-        <origin xyz="0 0 ${elem_length_main}" rpy="0 0 0"/>
-        <parent link="element_${elem_num-1}"/>
-        <child  link="element_${elem_num}"/>
-      </joint>
-    </xacro:if>
-  </xacro:macro>
-  <!-- Interior chain -->
-  <xacro:generate_cable elem_num="${num_elements}" />
-  <!-- Endcaps -->
-  <xacro:cable_element elem_name="element_first"
-                       elem_length="${elem_length_ends}"
-                       elem_mass="${elem_mass_ends}"/>
-  <xacro:cable_element elem_name="element_last"
-                       elem_length="${elem_length_ends}"
-                       elem_mass="${elem_mass_ends}"/>
-  <!-- First to element_1 -->
-  <joint name="joint_0_to_1" type="continuous">
-    <axis xyz="0 1 0">
-      <!-- <limit effort="${joint_effort}" velocity="${joint_velocity}"/> -->
-      <dynamics damping="${joint_damping}" friction="${joint_friction}"/>
-    </axis>
-    <origin xyz="0 0 ${elem_length_ends}" rpy="0 0 0"/>
-    <parent link="element_first"/>
-    <child  link="element_1"/>
-  </joint>
-  <!-- Last interior to endcap -->
-  <joint name="joint_${num_elements}_to_${num_elements+1}" type="continuous">
-    <axis xyz="0 1 0">
-      <!-- <limit effort="${joint_effort}" velocity="${joint_velocity}"/> -->
-      <dynamics damping="${joint_damping}" friction="${joint_friction}"/>
-    </axis>
-    <origin xyz="0 0 ${elem_length_main}" rpy="0 0 0"/>
-    <parent link="element_${num_elements}"/>
-    <child  link="element_last"/>
-  </joint>
+    <!-- Xacro to generate cable SDF -->
+    <!-- Note: need to manually find and replace all references to 'revolute'
+    with 'universal' in final SDF to get better cable. This also involves adding in a second axis.
+    These changes are now all defined in generate_sdf.sh-->
+    <!-- Define properties -->
+    <!-- <xacro:property name="dist_connect_points" value="1.5475" />  -->
+    <xacro:property name="cable_radius" value="${cable_radius}" />
+    <xacro:property name="cable_mass" value="${cable_mass}" />
+    <xacro:property name="cable_length" value="${cable_length}" />
+    <xacro:property name="num_elements" value="${num_elements}" />
+    <xacro:property name="elem_length_ends" value="${elem_length_ends}" />
+    <xacro:property name="elem_mass_ends" value="${elem_mass_ends}" />
+    <!-- Joint properties -->
+    <xacro:property name="joint_friction" value="${joint_friction}" />
+    <xacro:property name="joint_damping" value="${joint_damping}" />
+    <!-- Calculations -->
+    <xacro:property name="elem_mass_main" value="${cable_mass/num_elements}" />
+    <xacro:property name="ang_e" value="${pi/num_elements}"/>
+    <xacro:property name="ang_i" value="${pi - ang_e}"/>
+    <xacro:property name="elem_length_main" value="${cable_length/num_elements}"/>
+    <xacro:property name="dist_connect_points" value="${elem_length_main/sin(pi/(2*num_elements))}"/>
+    <!-- Define link macro -->
+    <xacro:macro name="cable_element" params="elem_name elem_length elem_mass">
+        <link name="${elem_name}">
+            <inertial>
+                <origin xyz="${elem_length/2} 0 0" rpy="0 ${pi/2} 0" />
+                <mass value="${elem_mass}"/>
+                <inertia ixx="${1/12*elem_mass*(3*cable_radius**2 + elem_length**2)}" ixy="0" ixz="0" iyy="${1/12*elem_mass*(3*cable_radius**2 + elem_length**2)}" iyz="0" izz="${1/2*elem_mass*(cable_radius**2)}" />
+            </inertial>
+            <visual>
+                <origin xyz="${elem_length/2} 0 0" rpy="0 ${pi/2} 0" />
+                <geometry>
+                    <cylinder length="${elem_length}" radius="${cable_radius}"/>
+                </geometry>
+            </visual>
+            <!-- <collision>
+                <origin xyz="${elem_length/2} 0 0" rpy="0 ${pi/2} 0" />
+                <geometry>
+                    <cylinder length="${elem_length}" radius="${cable_radius}"/> 0.0001
+                </geometry>
+            </collision> -->
+        </link>
+    </xacro:macro>
+    <!-- Recursive loop to generate multiple elements and joints for said elements -->
+    <xacro:macro name="generate_cable" params="elem_num">
+        <!-- Generate elements and recurse-->
+        <xacro:cable_element elem_name="element_${elem_num}" elem_length="${elem_length_main}" elem_mass="${elem_mass_main}" />
+        <xacro:if value="${elem_num-1}">
+            <xacro:generate_cable elem_num="${elem_num-1}" />
+        </xacro:if>
+        <!-- Define joints -->
+        <xacro:if value="${elem_num-1 > 0}">
+            <joint name="joint_${elem_num-1}_to_${elem_num}" type="continuous">
+                <axis xyz="0. 1. 0."/>
+                <!-- <axis xyz="0. 1. 1."/> -->
+                <origin xyz="${elem_length_main} 0 0" rpy="0 ${-ang_e} 0"/>
+                <!-- <xacro:if value="${elem_num  == 1}">
+                    <origin xyz="${elem_length_main} 0 0" rpy="0 ${ang_i/2} 0"/>
+                </xacro:if>
+                <xacro:if value="${elem_num  == num_elements}">
+                    <origin xyz="${elem_length_main} 0 0" rpy="0 ${(pi-ang_e)/2} 0"/>
+                </xacro:if>
+                <xacro:if value="${(elem_num > 1) and (elem_num < num_elements)}">
+                    <origin xyz="${elem_length_main} 0 0" rpy="0 ${-ang_e} 0"/>
+                </xacro:if> -->
+                <parent link="element_${elem_num-1}"/>
+                <child link="element_${elem_num}"/>
+                <dynamics damping="${joint_damping}" friction="${joint_friction}"/>
+            </joint>
+        </xacro:if>
+    </xacro:macro>
+    <!-- Call recursive loop to generate cable -->
+    <xacro:generate_cable elem_num="${num_elements}" />
+    <!-- Add start and end elements and joints-->
+    <xacro:cable_element elem_name="element_first" elem_length="${elem_length_ends}" elem_mass="${elem_mass_ends}" />
+    <xacro:cable_element elem_name="element_last" elem_length="${elem_length_ends}" elem_mass="${elem_mass_ends}" />
+    <joint name="joint_0_to_1" type="continuous">
+        <axis xyz="0. 1. 0."/>
+        <origin xyz="${elem_length_ends} 0 0" rpy="0 ${ang_i/2} 0"/>
+        <parent link="element_first"/>
+        <child link="element_1"/>
+        <dynamics damping="${joint_damping}" friction="${joint_friction}"/>
+    </joint>
+    <joint name="joint_${num_elements}_to_${num_elements+1}" type="continuous">
+        <axis xyz="0. 1. 0."/>
+        <origin xyz="${elem_length_main} 0 0" rpy="0 ${(pi-ang_e)/2} 0"/>
+        <parent link="element_${num_elements}"/>
+        <child link="element_last"/>
+        <dynamics damping="${joint_damping}" friction="${joint_friction}"/>
+    </joint>
 </robot>

Commit message: Prior to num_elements conversion test

File: Tools/simulation/gz/models/tether_2m/model.urdf (robot description, URDF)
Before this commit: robot tether_2m, 31 links, 30 joints
Links:
- removed link element_26
- removed link element_27
- removed link element_28
- removed link element_29
- link element_1: mass 0.0006896551724137932 -> 0.0008; geometry visual cylinder length=0.09684 radius=0.0031
- link element_10: mass 0.0006896551724137932 -> 0.0008; geometry visual cylinder length=0.09684 radius=0.0031
- link element_11: mass 0.0006896551724137932 -> 0.0008; geometry visual cylinder length=0.09684 radius=0.0031
- link element_12: mass 0.0006896551724137932 -> 0.0008; geometry visual cylinder length=0.09684 radius=0.0031
- link element_13: mass 0.0006896551724137932 -> 0.0008; geometry visual cylinder length=0.09684 radius=0.0031
- link element_14: mass 0.0006896551724137932 -> 0.0008; geometry visual cylinder length=0.09684 radius=0.0031
- link element_15: mass 0.0006896551724137932 -> 0.0008; geometry visual cylinder length=0.09684 radius=0.0031
- link element_16: mass 0.0006896551724137932 -> 0.0008; geometry visual cylinder length=0.09684 radius=0.0031
- link element_17: mass 0.0006896551724137932 -> 0.0008; geometry visual cylinder length=0.09684 radius=0.0031
- link element_18: mass 0.0006896551724137932 -> 0.0008; geometry visual cylinder length=0.09684 radius=0.0031
- link element_19: mass 0.0006896551724137932 -> 0.0008; geometry visual cylinder length=0.09684 radius=0.0031
- link element_2: mass 0.0006896551724137932 -> 0.0008; geometry visual cylinder length=0.09684 radius=0.0031
- link element_20: mass 0.0006896551724137932 -> 0.0008; geometry visual cylinder length=0.09684 radius=0.0031
- link element_21: mass 0.0006896551724137932 -> 0.0008; geometry visual cylinder length=0.09684 radius=0.0031
- link element_22: mass 0.0006896551724137932 -> 0.0008; geometry visual cylinder length=0.09684 radius=0.0031
- link element_23: mass 0.0006896551724137932 -> 0.0008; geometry visual cylinder length=0.09684 radius=0.0031
- link element_24: mass 0.0006896551724137932 -> 0.0008; geometry visual cylinder length=0.09684 radius=0.0031
- link element_25: mass 0.0006896551724137932 -> 0.0008; geometry visual cylinder length=0.09684 radius=0.0031
- link element_3: mass 0.0006896551724137932 -> 0.0008; geometry visual cylinder length=0.09684 radius=0.0031
- link element_4: mass 0.0006896551724137932 -> 0.0008; geometry visual cylinder length=0.09684 radius=0.0031
- link element_5: mass 0.0006896551724137932 -> 0.0008; geometry visual cylinder length=0.09684 radius=0.0031
- link element_6: mass 0.0006896551724137932 -> 0.0008; geometry visual cylinder length=0.09684 radius=0.0031
- link element_7: mass 0.0006896551724137932 -> 0.0008; geometry visual cylinder length=0.09684 radius=0.0031
- link element_8: mass 0.0006896551724137932 -> 0.0008; geometry visual cylinder length=0.09684 radius=0.0031
- link element_9: mass 0.0006896551724137932 -> 0.0008; geometry visual cylinder length=0.09684 radius=0.0031
Joints:
- removed joint joint_26_to_27
- removed joint joint_27_to_28
- removed joint joint_28_to_29
- removed joint joint_29_to_30
- joint joint_0_to_1: origin xyz=0.0001 0 0 rpy=0 1.5166309362157622 0 -> xyz=0.0001 0 0 rpy=0 1.5079644737231006 0
- joint joint_10_to_11: origin xyz=0.08348275862068964 0 0 rpy=0 -0.10833078115826873 0 -> xyz=0.09684 0 0 rpy=0 -0.12566370614359174 0
- joint joint_11_to_12: origin xyz=0.08348275862068964 0 0 rpy=0 -0.10833078115826873 0 -> xyz=0.09684 0 0 rpy=0 -0.12566370614359174 0
- joint joint_12_to_13: origin xyz=0.08348275862068964 0 0 rpy=0 -0.10833078115826873 0 -> xyz=0.09684 0 0 rpy=0 -0.12566370614359174 0
- joint joint_13_to_14: origin xyz=0.08348275862068964 0 0 rpy=0 -0.10833078115826873 0 -> xyz=0.09684 0 0 rpy=0 -0.12566370614359174 0
- joint joint_14_to_15: origin xyz=0.08348275862068964 0 0 rpy=0 -0.10833078115826873 0 -> xyz=0.09684 0 0 rpy=0 -0.12566370614359174 0
- joint joint_15_to_16: origin xyz=0.08348275862068964 0 0 rpy=0 -0.10833078115826873 0 -> xyz=0.09684 0 0 rpy=0 -0.12566370614359174 0
- joint joint_16_to_17: origin xyz=0.08348275862068964 0 0 rpy=0 -0.10833078115826873 0 -> xyz=0.09684 0 0 rpy=0 -0.12566370614359174 0
- joint joint_17_to_18: origin xyz=0.08348275862068964 0 0 rpy=0 -0.10833078115826873 0 -> xyz=0.09684 0 0 rpy=0 -0.12566370614359174 0
- joint joint_18_to_19: origin xyz=0.08348275862068964 0 0 rpy=0 -0.10833078115826873 0 -> xyz=0.09684 0 0 rpy=0 -0.12566370614359174 0
- joint joint_19_to_20: origin xyz=0.08348275862068964 0 0 rpy=0 -0.10833078115826873 0 -> xyz=0.09684 0 0 rpy=0 -0.12566370614359174 0
- joint joint_1_to_2: origin xyz=0.08348275862068964 0 0 rpy=0 -0.10833078115826873 0 -> xyz=0.09684 0 0 rpy=0 -0.12566370614359174 0
- joint joint_20_to_21: origin xyz=0.08348275862068964 0 0 rpy=0 -0.10833078115826873 0 -> xyz=0.09684 0 0 rpy=0 -0.12566370614359174 0
- joint joint_21_to_22: origin xyz=0.08348275862068964 0 0 rpy=0 -0.10833078115826873 0 -> xyz=0.09684 0 0 rpy=0 -0.12566370614359174 0
- joint joint_22_to_23: origin xyz=0.08348275862068964 0 0 rpy=0 -0.10833078115826873 0 -> xyz=0.09684 0 0 rpy=0 -0.12566370614359174 0
- joint joint_23_to_24: origin xyz=0.08348275862068964 0 0 rpy=0 -0.10833078115826873 0 -> xyz=0.09684 0 0 rpy=0 -0.12566370614359174 0
- joint joint_24_to_25: origin xyz=0.08348275862068964 0 0 rpy=0 -0.10833078115826873 0 -> xyz=0.09684 0 0 rpy=0 -0.12566370614359174 0
- joint joint_25_to_26: child element_26 -> element_last; origin xyz=0.08348275862068964 0 0 rpy=0 -0.10833078115826873 0 -> xyz=0.09684 0 0 rpy=0 1.5079644737231006 0
- joint joint_2_to_3: origin xyz=0.08348275862068964 0 0 rpy=0 -0.10833078115826873 0 -> xyz=0.09684 0 0 rpy=0 -0.12566370614359174 0
- joint joint_3_to_4: origin xyz=0.08348275862068964 0 0 rpy=0 -0.10833078115826873 0 -> xyz=0.09684 0 0 rpy=0 -0.12566370614359174 0
- joint joint_4_to_5: origin xyz=0.08348275862068964 0 0 rpy=0 -0.10833078115826873 0 -> xyz=0.09684 0 0 rpy=0 -0.12566370614359174 0
- joint joint_5_to_6: origin xyz=0.08348275862068964 0 0 rpy=0 -0.10833078115826873 0 -> xyz=0.09684 0 0 rpy=0 -0.12566370614359174 0
- joint joint_6_to_7: origin xyz=0.08348275862068964 0 0 rpy=0 -0.10833078115826873 0 -> xyz=0.09684 0 0 rpy=0 -0.12566370614359174 0
- joint joint_7_to_8: origin xyz=0.08348275862068964 0 0 rpy=0 -0.10833078115826873 0 -> xyz=0.09684 0 0 rpy=0 -0.12566370614359174 0
- joint joint_8_to_9: origin xyz=0.08348275862068964 0 0 rpy=0 -0.10833078115826873 0 -> xyz=0.09684 0 0 rpy=0 -0.12566370614359174 0
- joint joint_9_to_10: origin xyz=0.08348275862068964 0 0 rpy=0 -0.10833078115826873 0 -> xyz=0.09684 0 0 rpy=0 -0.12566370614359174 0

File: Tools/simulation/gz/models/tether_2m/model.xacro (robot description, xacro)
@@ -10,10 +10,10 @@
     <xacro:property name="cable_mass" value="0.02" />
     <xacro:property name="cable_length" value="2.421" />
-    <xacro:property name="num_elements" value="29" />
+    <xacro:property name="num_elements" value="25" />
     <xacro:property name="elem_length_ends" value="0.0001" />
     <xacro:property name="elem_mass_ends" value="0.0001" />
     <!-- Joint properties -->
-    <xacro:property name="joint_friction" value="0.0" />
-    <xacro:property name="joint_damping" value="0.0025" />
+    <xacro:property name="joint_friction" value="0" />
+    <xacro:property name="joint_damping" value="0.002" />
     <!-- Calculations -->
     <xacro:property name="elem_mass_main" value="${cable_mass/num_elements}" />
@@ -68,10 +68,10 @@
                 <parent link="element_${elem_num-1}"/>
                 <child link="element_${elem_num}"/>
-                <dynamics damping="0.0025" friction="0.0"/>
+                <dynamics damping="0.002" friction="0"/>
             </joint>
         </xacro:if>
     </xacro:macro>
     <!-- Call recursive loop to generate cable -->
-    <xacro:generate_cable elem_num="29" />
+    <xacro:generate_cable elem_num="25" />
     <!-- Add start and end elements and joints-->
     <xacro:cable_element elem_name="element_first" elem_length="0.0001" elem_mass="0.0001" />
@@ -82,12 +82,12 @@
         <parent link="element_first"/>
         <child link="element_1"/>
-        <dynamics damping="0.0025" friction="0.0"/>
+        <dynamics damping="0.002" friction="0"/>
     </joint>
-    <joint name="joint_29_to_${num_elements+1}" type="continuous">
+    <joint name="joint_25_to_${num_elements+1}" type="continuous">
         <axis xyz="0. 1. 0."/>
         <origin xyz="${elem_length_main} 0 0" rpy="0 ${(pi-ang_e)/2} 0"/>
-        <parent link="element_29"/>
+        <parent link="element_25"/>
         <child link="element_last"/>
-        <dynamics damping="0.0025" friction="0.0"/>
+        <dynamics damping="0.002" friction="0"/>
     </joint>
 </robot>
