Commit message: Pre-publish

File: Tools/simulation/gz/models/tether_2m/model.urdf (robot description, URDF)
Before this commit: robot tether_2m, 27 links, 26 joints
Links:
- removed link element_16
- removed link element_17
- removed link element_18
- removed link element_19
- removed link element_20
- removed link element_21
- removed link element_22
- removed link element_23
- removed link element_24
- removed link element_25
- link element_1: mass 0.0008 -> 0.0013333333333333333; geometry visual cylinder length=0.1614 radius=0.0031
- link element_10: mass 0.0008 -> 0.0013333333333333333; geometry visual cylinder length=0.1614 radius=0.0031
- link element_11: mass 0.0008 -> 0.0013333333333333333; geometry visual cylinder length=0.1614 radius=0.0031
- link element_12: mass 0.0008 -> 0.0013333333333333333; geometry visual cylinder length=0.1614 radius=0.0031
- link element_13: mass 0.0008 -> 0.0013333333333333333; geometry visual cylinder length=0.1614 radius=0.0031
- link element_14: mass 0.0008 -> 0.0013333333333333333; geometry visual cylinder length=0.1614 radius=0.0031
- link element_15: mass 0.0008 -> 0.0013333333333333333; geometry visual cylinder length=0.1614 radius=0.0031
- link element_2: mass 0.0008 -> 0.0013333333333333333; geometry visual cylinder length=0.1614 radius=0.0031
- link element_3: mass 0.0008 -> 0.0013333333333333333; geometry visual cylinder length=0.1614 radius=0.0031
- link element_4: mass 0.0008 -> 0.0013333333333333333; geometry visual cylinder length=0.1614 radius=0.0031
- link element_5: mass 0.0008 -> 0.0013333333333333333; geometry visual cylinder length=0.1614 radius=0.0031
- link element_6: mass 0.0008 -> 0.0013333333333333333; geometry visual cylinder length=0.1614 radius=0.0031
- link element_7: mass 0.0008 -> 0.0013333333333333333; geometry visual cylinder length=0.1614 radius=0.0031
- link element_8: mass 0.0008 -> 0.0013333333333333333; geometry visual cylinder length=0.1614 radius=0.0031
- link element_9: mass 0.0008 -> 0.0013333333333333333; geometry visual cylinder length=0.1614 radius=0.0031
Joints:
- removed joint joint_16_to_17
- removed joint joint_17_to_18
- removed joint joint_18_to_19
- removed joint joint_19_to_20
- removed joint joint_20_to_21
- removed joint joint_21_to_22
- removed joint joint_22_to_23
- removed joint joint_23_to_24
- removed joint joint_24_to_25
- removed joint joint_25_to_26
- joint joint_0_to_1: origin xyz=0.0001 0 0 rpy=0 1.5079644737231006 0 -> xyz=0.0001 0 0 rpy=0 1.4660765716752369 0
- joint joint_10_to_11: origin xyz=0.09684 0 0 rpy=0 -0.12566370614359174 0 -> xyz=0.1614 0 0 rpy=0 -0.20943951023931953 0
- joint joint_11_to_12: origin xyz=0.09684 0 0 rpy=0 -0.12566370614359174 0 -> xyz=0.1614 0 0 rpy=0 -0.20943951023931953 0
- joint joint_12_to_13: origin xyz=0.09684 0 0 rpy=0 -0.12566370614359174 0 -> xyz=0.1614 0 0 rpy=0 -0.20943951023931953 0
- joint joint_13_to_14: origin xyz=0.09684 0 0 rpy=0 -0.12566370614359174 0 -> xyz=0.1614 0 0 rpy=0 -0.20943951023931953 0
- joint joint_14_to_15: origin xyz=0.09684 0 0 rpy=0 -0.12566370614359174 0 -> xyz=0.1614 0 0 rpy=0 -0.20943951023931953 0
- joint joint_15_to_16: child element_16 -> element_last; origin xyz=0.09684 0 0 rpy=0 -0.12566370614359174 0 -> xyz=0.1614 0 0 rpy=0 1.4660765716752369 0
- joint joint_1_to_2: origin xyz=0.09684 0 0 rpy=0 -0.12566370614359174 0 -> xyz=0.1614 0 0 rpy=0 -0.20943951023931953 0
- joint joint_2_to_3: origin xyz=0.09684 0 0 rpy=0 -0.12566370614359174 0 -> xyz=0.1614 0 0 rpy=0 -0.20943951023931953 0
- joint joint_3_to_4: origin xyz=0.09684 0 0 rpy=0 -0.12566370614359174 0 -> xyz=0.1614 0 0 rpy=0 -0.20943951023931953 0
- joint joint_4_to_5: origin xyz=0.09684 0 0 rpy=0 -0.12566370614359174 0 -> xyz=0.1614 0 0 rpy=0 -0.20943951023931953 0
- joint joint_5_to_6: origin xyz=0.09684 0 0 rpy=0 -0.12566370614359174 0 -> xyz=0.1614 0 0 rpy=0 -0.20943951023931953 0
- joint joint_6_to_7: origin xyz=0.09684 0 0 rpy=0 -0.12566370614359174 0 -> xyz=0.1614 0 0 rpy=0 -0.20943951023931953 0
- joint joint_7_to_8: origin xyz=0.09684 0 0 rpy=0 -0.12566370614359174 0 -> xyz=0.1614 0 0 rpy=0 -0.20943951023931953 0
- joint joint_8_to_9: origin xyz=0.09684 0 0 rpy=0 -0.12566370614359174 0 -> xyz=0.1614 0 0 rpy=0 -0.20943951023931953 0
- joint joint_9_to_10: origin xyz=0.09684 0 0 rpy=0 -0.12566370614359174 0 -> xyz=0.1614 0 0 rpy=0 -0.20943951023931953 0

File: Tools/simulation/gz/models/tether_2m/model.xacro (robot description, xacro)
@@ -10,5 +10,5 @@
     <xacro:property name="cable_mass" value="0.02" />
     <xacro:property name="cable_length" value="2.421" />
-    <xacro:property name="num_elements" value="25" />
+    <xacro:property name="num_elements" value="15" />
     <xacro:property name="elem_length_ends" value="0.0001" />
     <xacro:property name="elem_mass_ends" value="0.0001" />
@@ -73,5 +73,5 @@
     </xacro:macro>
     <!-- Call recursive loop to generate cable -->
-    <xacro:generate_cable elem_num="25" />
+    <xacro:generate_cable elem_num="15" />
     <!-- Add start and end elements and joints-->
     <xacro:cable_element elem_name="element_first" elem_length="0.0001" elem_mass="0.0001" />
@@ -84,8 +84,8 @@
         <dynamics damping="0.002" friction="0"/>
     </joint>
-    <joint name="joint_25_to_${num_elements+1}" type="continuous">
+    <joint name="joint_15_to_${num_elements+1}" type="continuous">
         <axis xyz="0. 1. 0."/>
         <origin xyz="${elem_length_main} 0 0" rpy="0 ${(pi-ang_e)/2} 0"/>
-        <parent link="element_25"/>
+        <parent link="element_15"/>
         <child link="element_last"/>
         <dynamics damping="0.002" friction="0"/>
