Commit message: Updated plugin names in world, ensure world sdf is v1.10

File: Tools/simulation/gz/models/tether_2m/model.xacro (robot description, xacro)
@@ -14,6 +14,6 @@
     <xacro:property name="elem_mass_ends" value="0.0001" />
     <!-- Joint properties -->
-    <xacro:property name="joint_friction" value="0" />
-    <xacro:property name="joint_damping" value="0.0005" />
+    <xacro:property name="joint_friction" value="0.0" />
+    <xacro:property name="joint_damping" value="0.0025" />
     <!-- Calculations -->
     <xacro:property name="elem_mass_main" value="${cable_mass/num_elements}" />
@@ -68,5 +68,5 @@
                 <parent link="element_${elem_num-1}"/>
                 <child link="element_${elem_num}"/>
-                <dynamics damping="0.0005" friction="0"/>
+                <dynamics damping="0.0025" friction="0.0"/>
             </joint>
         </xacro:if>
@@ -82,5 +82,5 @@
         <parent link="element_first"/>
         <child link="element_1"/>
-        <dynamics damping="0.0005" friction="0"/>
+        <dynamics damping="0.0025" friction="0.0"/>
     </joint>
     <joint name="joint_29_to_${num_elements+1}" type="continuous">
@@ -89,5 +89,5 @@
         <parent link="element_29"/>
         <child link="element_last"/>
-        <dynamics damping="0.0005" friction="0"/>
+        <dynamics damping="0.0025" friction="0.0"/>
     </joint>
 </robot>

Commit message: Updated cable params

File: Tools/simulation/gz/models/tether_2m/model.xacro (robot description, xacro)
@@ -15,5 +15,5 @@
     <!-- Joint properties -->
     <xacro:property name="joint_friction" value="0" />
-    <xacro:property name="joint_damping" value="0.002" />
+    <xacro:property name="joint_damping" value="0.01" />
     <!-- Calculations -->
     <xacro:property name="elem_mass_main" value="${cable_mass/num_elements}" />
@@ -68,5 +68,5 @@
                 <parent link="element_${elem_num-1}"/>
                 <child link="element_${elem_num}"/>
-                <dynamics damping="0.002" friction="0"/>
+                <dynamics damping="0.01" friction="0"/>
             </joint>
         </xacro:if>
@@ -82,5 +82,5 @@
         <parent link="element_first"/>
         <child link="element_1"/>
-        <dynamics damping="0.002" friction="0"/>
+        <dynamics damping="0.01" friction="0"/>
     </joint>
     <joint name="joint_15_to_${num_elements+1}" type="continuous">
@@ -89,5 +89,5 @@
         <parent link="element_15"/>
         <child link="element_last"/>
-        <dynamics damping="0.002" friction="0"/>
+        <dynamics damping="0.01" friction="0"/>
     </joint>
 </robot>
